File: classic48/classic48.kicad_pcb (KiCad board)
At the start: 2 copper layers, 3.4 x 3 mm, 75 parts, among them SW1 Switch, SW10 Switch, SW11 Switch, SW12 Switch, SW13 Switch, SW14 Switch, SW15 Switch, SW16 Switch, SW17 Switch, SW18 Switch, SW19 Switch, SW2 Switch, SW20 Switch, SW21 Switch, SW22 Switch, SW23 Switch, SW24 Switch, SW3 Switch, SW4 Switch, SW5 Switch, SW6 Switch, SW7 Switch, SW8 Switch, SW9 Switch, U1 RP2040_Pro_Micro, U2 TRRS

Commit message: feat: finish tracks
Parts:
- moved U1 8.79 mm to (37.4, 39.8)
Connections:
- U1 pad 15: Row 3 Left -> Col 5 Left
- U1 pad 16: Row 2 Left -> Col 4 Left
- U1 pad 17: Row 1 Left -> Col 3 Left
- U1 pad 18: Row 0 Left -> Col 2 Left
- U1 pad 19: Col 5 Left -> Col 1 Left
- U1 pad 20: Col 4 Left -> Col 0 Left
- U1 pad 21: Col 3 Left -> Row 3 Left
- U1 pad 22: Col 2 Left -> Row 2 Left
- U1 pad 23: Col 1 Left -> Row 1 Left
- U1 pad 24: Col 0 Left -> Row 0 Left
Routing:
- net Col 5 Left: track 0.00 -> 196.1 mm, vias 0 -> 4
- net Col 4 Left: track 0.00 -> 176.3 mm, vias 0 -> 4
- net Col 3 Left: track 0.00 -> 153.5 mm, vias 0 -> 4
- net Col 2 Left: track 0.00 -> 136.4 mm, vias 0 -> 4
- net Row 3 Left: track 0.00 -> 135.2 mm
- net Row 2 Left: track 0.00 -> 119.3 mm
- net Col 1 Left: track 0.00 -> 116.5 mm, vias 0 -> 4
- net Row 0 Left: track 0.00 -> 111.8 mm
- net Row 1 Left: track 0.00 -> 108.3 mm, vias 0 -> 2
- net Col 0 Left: track 0.00 -> 86.8 mm, vias 0 -> 6
- net GND Left: track 507.9 -> 496.8 mm
- net Serial data left: track 130.9 -> 122.0 mm
- net 5V Left: track 496.9 -> 488.3 mm
- net LED Data Left: track 21.9 -> 14.1 mm
- net Net-(D24-A): track 0.00 -> 3.26 mm
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Other:
- board size 3.4 x 3 mm -> 144.6 x 71 mm
