File: classic48/classic48.kicad_pcb (KiCad board)
At the start: 2 copper layers, 135.8 x 69.8 mm, 75 parts, among them SW1 Switch, SW10 Switch, SW11 Switch, SW12 Switch, SW13 Switch, SW14 Switch, SW15 Switch, SW16 Switch, SW17 Switch, SW18 Switch, SW19 Switch, SW2 Switch, SW20 Switch, SW21 Switch, SW22 Switch, SW23 Switch, SW24 Switch, SW3 Switch, SW4 Switch, SW5 Switch, SW6 Switch, SW7 Switch, SW8 Switch, SW9 Switch, U1 RP2040_Pro_Micro, U2 TRRS

Commit message: feat: right switches positions
Parts:
- added D26: Diode_1N4148-SOD123, pjimenez:Diode_1N4148-SOD123, F.Cu at (339.0, 200.6)
- added D27: Diode_1N4148-SOD123, pjimenez:Diode_1N4148-SOD123, F.Cu at (339.0, 203.3)
- added D28: Diode_1N4148-SOD123, pjimenez:Diode_1N4148-SOD123, F.Cu at (339.0, 205.9)
- added D29: Diode_1N4148-SOD123, pjimenez:Diode_1N4148-SOD123, F.Cu at (339.0, 208.6)
- added D30: Diode_1N4148-SOD123, pjimenez:Diode_1N4148-SOD123, F.Cu at (339.0, 211.2)
- added D31: Diode_1N4148-SOD123, pjimenez:Diode_1N4148-SOD123, F.Cu at (339.0, 213.9)
- added D32: Diode_1N4148-SOD123, pjimenez:Diode_1N4148-SOD123, F.Cu at (339.0, 216.5)
- added D33: Diode_1N4148-SOD123, pjimenez:Diode_1N4148-SOD123, F.Cu at (339.0, 219.2)
- added D34: Diode_1N4148-SOD123, pjimenez:Diode_1N4148-SOD123, F.Cu at (339.0, 221.8)
- added D35: Diode_1N4148-SOD123, pjimenez:Diode_1N4148-SOD123, F.Cu at (345.8, 200.6)
- added D36: Diode_1N4148-SOD123, pjimenez:Diode_1N4148-SOD123, F.Cu at (345.8, 203.3)
- added D37: Diode_1N4148-SOD123, pjimenez:Diode_1N4148-SOD123, F.Cu at (345.8, 205.9)
- added D38: Diode_1N4148-SOD123, pjimenez:Diode_1N4148-SOD123, F.Cu at (345.8, 208.6)
- added D39: Diode_1N4148-SOD123, pjimenez:Diode_1N4148-SOD123, F.Cu at (345.8, 211.2)
- added D40: Diode_1N4148-SOD123, pjimenez:Diode_1N4148-SOD123, F.Cu at (345.8, 213.9)
- added D41: Diode_1N4148-SOD123, pjimenez:Diode_1N4148-SOD123, F.Cu at (345.8, 216.5)
- added D42: Diode_1N4148-SOD123, pjimenez:Diode_1N4148-SOD123, F.Cu at (345.8, 219.2)
- added D43: Diode_1N4148-SOD123, pjimenez:Diode_1N4148-SOD123, F.Cu at (345.8, 221.8)
- added D44: Diode_1N4148-SOD123, pjimenez:Diode_1N4148-SOD123, F.Cu at (352.6, 200.6)
- added D45: Diode_1N4148-SOD123, pjimenez:Diode_1N4148-SOD123, F.Cu at (352.6, 203.3)
- added D46: Diode_1N4148-SOD123, pjimenez:Diode_1N4148-SOD123, F.Cu at (352.6, 205.9)
- added D47: Diode_1N4148-SOD123, pjimenez:Diode_1N4148-SOD123, F.Cu at (352.6, 208.6)
- added D48: Diode_1N4148-SOD123, pjimenez:Diode_1N4148-SOD123, F.Cu at (352.6, 211.2)
- added D49: Diode_1N4148-SOD123, pjimenez:Diode_1N4148-SOD123, F.Cu at (352.6, 213.9)
- added D50: Diode_1N4148-SOD123, pjimenez:Diode_1N4148-SOD123, F.Cu at (352.6, 216.5)
- added LED25: LED_SK6812MINI-E, pjimenez:LED_SK6812-MINI-E, F.Cu at (339.4, 176.7)
- added LED26: LED_SK6812MINI-E, pjimenez:LED_SK6812-MINI-E, F.Cu at (339.4, 180.8)
- added LED27: LED_SK6812MINI-E, pjimenez:LED_SK6812-MINI-E, F.Cu at (339.4, 184.9)
- added LED28: LED_SK6812MINI-E, pjimenez:LED_SK6812-MINI-E, F.Cu at (339.4, 189.0)
- added LED29: LED_SK6812MINI-E, pjimenez:LED_SK6812-MINI-E, F.Cu at (339.4, 193.1)
- added LED30: LED_SK6812MINI-E, pjimenez:LED_SK6812-MINI-E, F.Cu at (339.4, 197.3)
- added LED31: LED_SK6812MINI-E, pjimenez:LED_SK6812-MINI-E, F.Cu at (347.3, 176.7)
- added LED32: LED_SK6812MINI-E, pjimenez:LED_SK6812-MINI-E, F.Cu at (347.3, 180.8)
- added LED33: LED_SK6812MINI-E, pjimenez:LED_SK6812-MINI-E, F.Cu at (347.3, 184.9)
- added LED34: LED_SK6812MINI-E, pjimenez:LED_SK6812-MINI-E, F.Cu at (347.3, 189.0)
- added LED35: LED_SK6812MINI-E, pjimenez:LED_SK6812-MINI-E, F.Cu at (347.3, 193.1)
- added LED36: LED_SK6812MINI-E, pjimenez:LED_SK6812-MINI-E, F.Cu at (347.3, 197.3)
- added LED37: LED_SK6812MINI-E, pjimenez:LED_SK6812-MINI-E, F.Cu at (355.1, 176.7)
- added LED38: LED_SK6812MINI-E, pjimenez:LED_SK6812-MINI-E, F.Cu at (355.1, 180.8)
- added LED39: LED_SK6812MINI-E, pjimenez:LED_SK6812-MINI-E, F.Cu at (355.1, 184.9)
- added LED40: LED_SK6812MINI-E, pjimenez:LED_SK6812-MINI-E, F.Cu at (355.1, 189.0)
- added LED41: LED_SK6812MINI-E, pjimenez:LED_SK6812-MINI-E, F.Cu at (355.1, 193.1)
- added LED42: LED_SK6812MINI-E, pjimenez:LED_SK6812-MINI-E, F.Cu at (355.1, 197.3)
- added LED43: LED_SK6812MINI-E, pjimenez:LED_SK6812-MINI-E, F.Cu at (363.0, 176.7)
- added LED44: LED_SK6812MINI-E, pjimenez:LED_SK6812-MINI-E, F.Cu at (363.0, 180.8)
- added LED45: LED_SK6812MINI-E, pjimenez:LED_SK6812-MINI-E, F.Cu at (363.0, 184.9)
- added LED46: LED_SK6812MINI-E, pjimenez:LED_SK6812-MINI-E, F.Cu at (363.0, 189.0)
- added LED47: LED_SK6812MINI-E, pjimenez:LED_SK6812-MINI-E, F.Cu at (363.0, 193.1)
- added LED48: LED_SK6812MINI-E, pjimenez:LED_SK6812-MINI-E, F.Cu at (363.0, 197.3)
- added SW25: Switch, pjimenez:Switch_ChocV1-hotswap, F.Cu at (57.0, 103.3)
- added SW26: Switch, pjimenez:Switch_ChocV1-hotswap, F.Cu at (75.0, 103.3)
- added SW27: Switch, pjimenez:Switch_ChocV1-hotswap, F.Cu at (93.0, 103.3)
- added SW28: Switch, pjimenez:Switch_ChocV1-hotswap, F.Cu at (111.0, 103.3)
- added SW29: Switch, pjimenez:Switch_ChocV1-hotswap, F.Cu at (129.0, 103.3)
- added SW30: Switch, pjimenez:Switch_ChocV1-hotswap, F.Cu at (147.0, 103.3)
- added SW31: Switch, pjimenez:Switch_ChocV1-hotswap, F.Cu at (57.0, 120.3)
- added SW32: Switch, pjimenez:Switch_ChocV1-hotswap, F.Cu at (75.0, 120.3)
- added SW33: Switch, pjimenez:Switch_ChocV1-hotswap, F.Cu at (93.0, 120.3)
- added SW34: Switch, pjimenez:Switch_ChocV1-hotswap, F.Cu at (111.0, 120.3)
- added SW35: Switch, pjimenez:Switch_ChocV1-hotswap, F.Cu at (129.0, 120.3)
- added SW36: Switch, pjimenez:Switch_ChocV1-hotswap, F.Cu at (147.0, 120.3)
- added SW37: Switch, pjimenez:Switch_ChocV1-hotswap, F.Cu at (57.0, 137.3)
- added SW38: Switch, pjimenez:Switch_ChocV1-hotswap, F.Cu at (75.0, 137.3)
- added SW39: Switch, pjimenez:Switch_ChocV1-hotswap, F.Cu at (93.0, 137.3)
- added SW40: Switch, pjimenez:Switch_ChocV1-hotswap, F.Cu at (111.0, 137.3)
- added SW41: Switch, pjimenez:Switch_ChocV1-hotswap, F.Cu at (129.0, 137.3)
- added SW42: Switch, pjimenez:Switch_ChocV1-hotswap, F.Cu at (147.0, 137.3)
- added SW43: Switch, pjimenez:Switch_ChocV1-hotswap, F.Cu at (57.0, 154.3)
- added SW44: Switch, pjimenez:Switch_ChocV1-hotswap, F.Cu at (75.0, 154.3)
- added SW45: Switch, pjimenez:Switch_ChocV1-hotswap, F.Cu at (93.0, 154.3)
- added SW46: Switch, pjimenez:Switch_ChocV1-hotswap, F.Cu at (111.0, 154.3)
- added SW47: Switch, pjimenez:Switch_ChocV1-hotswap, F.Cu at (129.0, 154.3)
- added SW48: Switch, pjimenez:Switch_ChocV1-hotswap, F.Cu at (147.0, 154.3)
- added U3: RP2040_Pro_Micro, pjimenez:RP2040_Pro_Micro, F.Cu at (420.4, 154.9)
- added U4: TRRS, pjimenez:TRRS_PJ-320A, F.Cu at (359.5, 201.9)

Commit message: feat: LED and switch positions
Parts:
- D26, D27, D28, D29, D30, D31, D32, D33, D34, D35, D36, D37, D38, D39, D40, D41, D42, D43, D44, D45, D46, D47, D48, D49, D50: moved to B.Cu
- moved LED43 307.2 mm to (57.0, 149.6), turned to 180 degrees
- moved LED42 305.1 mm to (57.0, 132.6)
- moved LED30 299.1 mm to (57.0, 98.6)
- moved D44 297.2 mm to (58.6, 157.0)
- moved LED31 296.6 mm to (57.0, 115.6), turned to 180 degrees
- moved D26 295.9 mm to (58.6, 106.0)
- moved D32 295.6 mm to (58.6, 123.0)
- moved D38 295.3 mm to (58.6, 140.0)
- moved LED44 289.7 mm to (75.0, 149.6), turned to 180 degrees
- moved LED41 286.6 mm to (75.0, 132.6)
- moved LED29 280.8 mm to (75.0, 98.6)
- moved LED32 279.9 mm to (75.0, 115.6), turned to 180 degrees
- moved D27 279.9 mm to (76.6, 106.0)
- moved D45 279.9 mm to (76.6, 157.0)
- moved D33 279.5 mm to (76.6, 123.0)
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
Commit message: feat: position MCU and TRRS
Parts:
- moved U4 360.1 mm to (44.0, 97.7)
- moved U3 257.4 mm to (166.5, 112.6)
Changed lines of the file:
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@@
 	(footprint "pjimenez:RP2040_Pro_Micro"
 		(layer "F.Cu")
-		(at 420.385 154.915)
+		(at 166.49 112.58)
 		(property "Reference" "U3"
 			(at 0 -1.27 0)
@@
 	(footprint "pjimenez:TRRS_PJ-320A"
 		(layer "F.Cu")
-		(at 388.6 202.0875)
+		(at 44 97.688)
 		(property "Reference" "U4"
 			(at 0 14.2 0)

Commit message: feat: fully wired
Parts:
- turned LED36 to 180 degrees
Routing:
- net 5V Right: track 0.00 -> 509.5 mm, vias 0 -> 3
- net GND Right: track 0.00 -> 503.7 mm, vias 0 -> 2
- net Col 5 Right: track 0.00 -> 177.7 mm, vias 0 -> 2
- net Col 4 Right: track 0.00 -> 171.6 mm, vias 0 -> 5
- net Col 3 Right: track 0.00 -> 155.9 mm, vias 0 -> 5
- net Row 3 Right: track 0.00 -> 146.2 mm, vias 0 -> 1
- net Serial data Right: track 0.00 -> 143.1 mm, vias 0 -> 2
- net Col 2 Right: track 0.00 -> 138.0 mm, vias 0 -> 5
- net Row 2 Right: track 0.00 -> 131.9 mm
- net Row 0 Right: track 0.00 -> 124.4 mm
- net Col 1 Right: track 0.00 -> 124.1 mm, vias 0 -> 5
- net Row 1 Right: track 0.00 -> 123.2 mm, vias 0 -> 1
- net Col 0 Right: track 0.00 -> 109.5 mm, vias 0 -> 5
- net LED data Right: track 0.00 -> 29.1 mm
- net Net-(LED36-DOUT): track 0.00 -> 22.6 mm
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