File: classic48/classic48.kicad_pcb (KiCad board)
At the start: 2 copper layers, 135.8 x 69.8 mm, 150 parts, among them SW1 Switch, SW10 Switch, SW11 Switch, SW12 Switch, SW13 Switch, SW14 Switch, SW15 Switch, SW16 Switch, SW17 Switch, SW18 Switch, SW19 Switch, SW2 Switch, SW20 Switch, SW21 Switch, SW22 Switch, SW23 Switch, SW24 Switch, SW25 Switch, SW26 Switch, SW27 Switch, SW28 Switch, SW29 Switch, SW3 Switch, SW30 Switch, SW31 Switch, SW32 Switch, SW33 Switch, SW34 Switch, SW35 Switch, SW36 Switch, SW37 Switch, SW38 Switch, SW39 Switch, SW4 Switch, SW40 Switch, SW41 Switch, SW42 Switch, SW43 Switch, SW44 Switch, SW45 Switch, SW46 Switch, SW47 Switch, SW48 Switch, SW5 Switch, SW6 Switch, SW7 Switch, SW8 Switch, SW9 Switch, U1 RP2040_Pro_Micro, U2 TRRS, U3 RP2040_Pro_Micro, U4 TRRS

Commit message: wip: working on the cuts
Parts:
- moved SW37 136.9 mm to (179.3, 75.8)
- moved SW38 136.9 mm to (197.3, 75.8)
- moved SW39 136.9 mm to (215.3, 75.8)
- moved SW40 136.9 mm to (233.3, 75.8)
- moved SW41 136.9 mm to (251.3, 75.8)
- moved SW42 136.9 mm to (269.3, 75.8)
- moved SW43 136.9 mm to (179.3, 92.8)
- moved SW44 136.9 mm to (197.3, 92.8)
- moved SW45 136.9 mm to (215.3, 92.8)
- moved SW46 136.9 mm to (233.3, 92.8)
- moved SW47 136.9 mm to (251.3, 92.8)
- moved SW48 136.9 mm to (269.3, 92.8)
- moved D26 136.9 mm to (180.9, 44.5)
- moved D27 136.9 mm to (198.9, 44.5)
- moved D28 136.9 mm to (216.9, 44.5)
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Other:
- board size 135.8 x 69.8 mm -> 283.2 x 97.3 mm

Commit message: feat: add structure
Parts:
- moved U4 8.35 mm to (157.9, 36.0)
- moved D26 8.31 mm to (172.6, 44.2)
- moved D27 8.31 mm to (190.6, 44.2)
- moved D28 8.31 mm to (208.6, 44.2)
- moved D29 8.31 mm to (226.6, 44.2)
- moved D30 8.31 mm to (244.6, 44.2)
- moved D32 8.31 mm to (172.6, 61.2)
- moved D33 8.31 mm to (190.6, 61.2)
- moved D34 8.31 mm to (208.6, 61.2)
- moved D35 8.31 mm to (226.6, 61.2)
- moved D36 8.31 mm to (244.6, 61.2)
- moved D38 8.31 mm to (172.6, 78.2)
- moved D39 8.31 mm to (190.6, 78.2)
- moved D40 8.31 mm to (208.6, 78.2)
- moved D41 8.31 mm to (226.6, 78.2)
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Other:
- board size 283.2 x 97.3 mm -> 275.5 x 76 mm

Commit message: feat: add graphics
Parts:
- added G***: LOGO, pjimenez:hacker_emblem, F.Cu at (280.1, 91.6)
- added G***: LOGO, pjimenez:hacker_emblem, F.Cu at (25.4, 91.6)
Other:
- board text added: "https://github.com/pablojimenezmateo/classic48 V0"

Commit message: feat: fill zone and export
Routing:
- added copper zone on B.Cu, net (none)
- added copper zone on F.Cu, net (none)
Changed lines of the file:
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@@
 		(net 154)
 	)
+	(zone
+		(net 0)
+		(net_name "")
+		(layers "F&B.Cu")
+		(hatch edge 0.5)
+		(priority 1)
+		(connect_pads
+			(clearance 0.5)
+		)
+		(min_thickness 0.25)
+		(filled_areas_thickness no)
+		(fill yes
+			(thermal_gap 0.5)
+			(thermal_bridge_width 0.5)
+			(island_removal_mode 1)
+			(island_area_min 10)
+		)
+		(polygon
+			(pts
+				(xy 152.5 24) (xy 295 24) (xy 295 106) (xy 153 108)
+			)
+		)
+	)
+	(zone
+		(net 0)
+		(net_name "")
+		(layers "F&B.Cu")
+		(hatch edge 0.5)
+		(connect_pads
+			(clearance 0.5)
+		)
+		(min_thickness 0.25)
+		(filled_areas_thickness no)
+		(fill yes
+			(thermal_gap 0.5)
+			(thermal_bridge_width 0.5)
+			(island_removal_mode 1)
+			(island_area_min 10)
+		)
+		(polygon
+			(pts
+				(xy 14 23.5) (xy 152.5 24) (xy 153 108) (xy 12.5 108.5)
+			)
+		)
+	)
 )
